Commit message: sim 2.0

File: urdf/dock_station.urdf.xacro (robot description, xacro)
@@ -291,5 +291,5 @@
     <parent link="kapak2"/>
     <child link="inside_camera_link"/>
-    <origin xyz="0.57 0.05 0" rpy="0 0 -1.85"/>
+    <origin xyz="0.55 0.05 0" rpy="-1.5708 0 -1.9708"/>
   </joint>
   <gazebo reference="inside_camera_link">
